File: 02_MCU_Inputs_Debug.kicad_sch (KiCad schematic)
At the start: 20 parts, among them SW1 UP, SW2 DOWN, SW3 LEFT, SW4 RIGHT, SW5 START, U1 STM32G030K8T6

Commit message: Complete procurement BOM and document component review gates
Parts:
- C10, C12: value 100n / 10V X7R -> 100n / 50V X7R; MPN (none) -> C1608X7R1H104K080AA; Manufacturer (none) -> TDK
- C11: value 4.7u / 10V X7R -> 4.7u / 16V; MPN (none) -> GRM188Z71C475KE21D; Manufacturer (none) -> Murata Manufacturing
- R10, R11, R12, R13, R14, R15: value 10k -> 10k 1%; MPN (none) -> ERJ3EKF1002V; Manufacturer (none) -> Panasonic Industry
- SW1, SW2, SW3, SW4, SW5: Manufacturer (none) -> Alps Alpine
- U1: Manufacturer (none) -> STMicroelectronics
Changed lines of the file:
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@@
+        (font
+          (size 1.27 1.27)) hide))
+    (property "Manufacturer" "STMicroelectronics"
+      (at 101.6 106.68 0)
+      (effects
         (font
           (size 1.27 1.27)) hide))
@@
         (font
           (size 1.27 1.27))))
-    (property "Value" "100n / 10V X7R"
+    (property "Value" "100n / 50V X7R"
       (at 52.18 176.53 0)
       (effects
@@
         (font
           (size 1.27 1.27)) hide))
-    (property "Datasheet" ""
+    (property "Datasheet" "https://product.tdk.com/info/en/documents/chara_sheet/C1608X7R1H104K080AA.pdf"
       (at 43.18 175.26 0)
       (effects
         (font
           (size 1.27 1.27)) hide))
-    (property "MPN" ""
+    (property "MPN" "C1608X7R1H104K080AA"
+      (at 43.18 175.26 0)
+      (effects
+        (font
+          (size 1.27 1.27)) hide))
+    (property "Manufacturer" "TDK"
       (at 43.18 175.26 0)
       (effects
@@
         (font
           (size 1.27 1.27))))
-    (property "Value" "4.7u / 10V X7R"
+    (property "Value" "4.7u / 16V"
       (at 95.36 176.53 0)
       (effects
@@
         (font
           (size 1.27 1.27)) hide))
-    (property "Datasheet" ""
+    (property "Datasheet" "https://search.murata.co.jp/Ceramy/image/img/A01X/G101/ENG/GRM188Z71C475KE21-01A.pdf"
       (at 86.36 175.26 0)
       (effects
         (font
           (size 1.27 1.27)) hide))
-    (property "MPN" ""
+    (property "MPN" "GRM188Z71C475KE21D"
+      (at 86.36 175.26 0)
+      (effects
+        (font
+          (size 1.27 1.27)) hide))
+    (property "Manufacturer" "Murata Manufacturing"
       (at 86.36 175.26 0)
       (effects
@@
         (font
           (size 1.27 1.27))))
-    (property "Value" "10k"
+    (property "Value" "10k 1%"
       (at 141.08 176.53 0)
       (effects
@@
         (font
           (size 1.27 1.27)) hide))
-    (property "Datasheet" ""
+    (property "Datasheet" "https://industrial.panasonic.com/cdbs/www-data/pdf/RDA0000/AOA0000C304.pdf"
       (at 132.08 175.26 0)
       (effects
         (font
           (size 1.27 1.27)) hide))
-    (property "MPN" ""
+    (property "MPN" "ERJ3EKF1002V"
+      (at 132.08 175.26 0)
+      (effects
+        (font
+          (size 1.27 1.27)) hide))
+    (property "Manufacturer" "Panasonic Industry"
       (at 132.08 175.26 0)
       (effects
@@
         (font
           (size 1.27 1.27))))
-    (property "Value" "100n / 10V X7R"
+    (property "Value" "100n / 50V X7R"
       (at 186.8 176.53 0)
       (effects
@@
         (font
           (size 1.27 1.27)) hide))
-    (property "Datasheet" ""
+    (property "Datasheet" "https://product.tdk.com/info/en/documents/chara_sheet/C1608X7R1H104K080AA.pdf"
       (at 177.8 175.26 0)
       (effects
         (font
           (size 1.27 1.27)) hide))
-    (property "MPN" ""
+    (property "MPN" "C1608X7R1H104K080AA"
+      (at 177.8 175.26 0)
+      (effects
+        (font
+          (size 1.27 1.27)) hide))
+    (property "Manufacturer" "TDK"
       (at 177.8 175.26 0)
       (effects
@@
         (font
           (size 1.27 1.27))))
-    (property "Value" "10k"
+    (property "Value" "10k 1%"
       (at 250.3 54.61 0)
       (effects
@@
         (font
           (size 1.27 1.27)) hide))
-    (property "Datasheet" ""
+    (property "Datasheet" "https://industrial.panasonic.com/cdbs/www-data/pdf/RDA0000/AOA0000C304.pdf"
       (at 241.3 53.34 0)
       (effects
         (font
           (size 1.27 1.27)) hide))
-    (property "MPN" ""
+    (property "MPN" "ERJ3EKF1002V"
+      (at 241.3 53.34 0)
+      (effects
+        (font
+          (size 1.27 1.27)) hide))
+    (property "Manufacturer" "Panasonic Industry"
       (at 241.3 53.34 0)
       (effects
@@
         (font
           (size 1.27 1.27)) hide))
-    (property "Datasheet" ""
+    (property "Datasheet" "https://tech.alpsalpine.com/cms.media/SKQGAB_KQG_719_EN_cc4e10226e.pdf"
       (at 327.66 60.96 0)
       (effects
@@
           (size 1.27 1.27)) hide))
     (property "MPN" "SKQGABE010"
+      (at 327.66 60.96 0)
+      (effects
+        (font
+          (size 1.27 1.27)) hide))
+    (property "Manufacturer" "Alps Alpine"
       (at 327.66 60.96 0)
       (effects
@@
         (font
           (size 1.27 1.27))))
-    (property "Value" "10k"
+    (property "Value" "10k 1%"
       (at 250.3 90.17 0)
       (effects
@@
         (font
           (size 1.27 1.27)) hide))
-    (property "Datasheet" ""
+    (property "Datasheet" "https://industrial.panasonic.com/cdbs/www-data/pdf/RDA0000/AOA0000C304.pdf"
       (at 241.3 88.9 0)
       (effects
         (font
           (size 1.27 1.27)) hide))
-    (property "MPN" ""
+    (property "MPN" "ERJ3EKF1002V"
+      (at 241.3 88.9 0)
+      (effects
+        (font
+          (size 1.27 1.27)) hide))
+    (property "Manufacturer" "Panasonic Industry"
       (at 241.3 88.9 0)
       (effects
@@
         (font
           (size 1.27 1.27)) hide))
-    (property "Datasheet" ""
+    (property "Datasheet" "https://tech.alpsalpine.com/cms.media/SKQGAB_KQG_719_EN_cc4e10226e.pdf"
       (at 327.66 96.52 0)
       (effects
@@
           (size 1.27 1.27)) hide))
     (property "MPN" "SKQGABE010"
+      (at 327.66 96.52 0)
+      (effects
+        (font
+          (size 1.27 1.27)) hide))
+    (property "Manufacturer" "Alps Alpine"
       (at 327.66 96.52 0)
       (effects
@@
         (font
           (size 1.27 1.27))))
-    (property "Value" "10k"
+    (property "Value" "10k 1%"
       (at 250.3 125.73 0)
       (effects
@@
         (font
           (size 1.27 1.27)) hide))
-    (property "Datasheet" ""
+    (property "Datasheet" "https://industrial.panasonic.com/cdbs/www-data/pdf/RDA0000/AOA0000C304.pdf"
       (at 241.3 124.46 0)
       (effects
         (font
           (size 1.27 1.27)) hide))
-    (property "MPN" ""
+    (property "MPN" "ERJ3EKF1002V"
+      (at 241.3 124.46 0)
+      (effects
+        (font
+          (size 1.27 1.27)) hide))
+    (property "Manufacturer" "Panasonic Industry"
       (at 241.3 124.46 0)
       (effects
@@
         (font
           (size 1.27 1.27)) hide))
-    (property "Datasheet" ""
+    (property "Datasheet" "https://tech.alpsalpine.com/cms.media/SKQGAB_KQG_719_EN_cc4e10226e.pdf"
       (at 327.66 132.08 0)
       (effects
@@
           (size 1.27 1.27)) hide))
     (property "MPN" "SKQGABE010"
+      (at 327.66 132.08 0)
+      (effects
+        (font
+          (size 1.27 1.27)) hide))
+    (property "Manufacturer" "Alps Alpine"
       (at 327.66 132.08 0)
       (effects
@@
         (font
           (size 1.27 1.27))))
-    (property "Value" "10k"
+    (property "Value" "10k 1%"
       (at 250.3 161.29 0)
       (effects
@@
         (font
           (size 1.27 1.27)) hide))
-    (property "Datasheet" ""
+    (property "Datasheet" "https://industrial.panasonic.com/cdbs/www-data/pdf/RDA0000/AOA0000C304.pdf"
       (at 241.3 160.02 0)
       (effects
         (font
           (size 1.27 1.27)) hide))
-    (property "MPN" ""
+    (property "MPN" "ERJ3EKF1002V"
+      (at 241.3 160.02 0)
+      (effects
+        (font
+          (size 1.27 1.27)) hide))
+    (property "Manufacturer" "Panasonic Industry"
       (at 241.3 160.02 0)
       (effects
@@
         (font
           (size 1.27 1.27)) hide))
-    (property "Datasheet" ""
+    (property "Datasheet" "https://tech.alpsalpine.com/cms.media/SKQGAB_KQG_719_EN_cc4e10226e.pdf"
       (at 327.66 167.64 0)
       (effects
@@
           (size 1.27 1.27)) hide))
     (property "MPN" "SKQGABE010"
+      (at 327.66 167.64 0)
+      (effects
+        (font
+          (size 1.27 1.27)) hide))
+    (property "Manufacturer" "Alps Alpine"
       (at 327.66 167.64 0)
       (effects
@@
         (font
           (size 1.27 1.27))))
-    (property "Value" "10k"
+    (property "Value" "10k 1%"
       (at 250.3 196.85 0)
       (effects
@@
         (font
           (size 1.27 1.27)) hide))
-    (property "Datasheet" ""
+    (property "Datasheet" "https://industrial.panasonic.com/cdbs/www-data/pdf/RDA0000/AOA0000C304.pdf"
       (at 241.3 195.58 0)
       (effects
         (font
           (size 1.27 1.27)) hide))
-    (property "MPN" ""
+    (property "MPN" "ERJ3EKF1002V"
+      (at 241.3 195.58 0)
+      (effects
+        (font
+          (size 1.27 1.27)) hide))
+    (property "Manufacturer" "Panasonic Industry"
       (at 241.3 195.58 0)
       (effects
@@
         (font
           (size 1.27 1.27)) hide))
-    (property "Datasheet" ""
+    (property "Datasheet" "https://tech.alpsalpine.com/cms.media/SKQGAB_KQG_719_EN_cc4e10226e.pdf"
       (at 327.66 203.2 0)
       (effects
@@
           (size 1.27 1.27)) hide))
     (property "MPN" "SKQGABE010"
+      (at 327.66 203.2 0)
+      (effects
+        (font
+          (size 1.27 1.27)) hide))
+    (property "Manufacturer" "Alps Alpine"
       (at 327.66 203.2 0)
       (effects
@@
         (font
           (size 1.27 1.27)) hide))
+    (property "Manufacturer" ""
+      (at 30.48 269.24 0)
+      (effects
+        (font
+          (size 1.27 1.27)) hide))
     (pin "1"
 )
@@
         (font
           (size 1.27 1.27)) hide))
+    (property "Manufacturer" ""
+      (at 66.04 269.24 0)
+      (effects
+        (font
+          (size 1.27 1.27)) hide))
     (pin "1"
 )
@@
         (font
           (size 1.27 1.27)) hide))
+    (property "Manufacturer" ""
+      (at 101.6 269.24 0)
+      (effects
+        (font
+          (size 1.27 1.27)) hide))
     (pin "1"
 )
@@
         (font
           (size 1.27 1.27)) hide))
+    (property "Manufacturer" ""
+      (at 137.16 269.24 0)
+      (effects
+        (font
+          (size 1.27 1.27)) hide))
     (pin "1"
 )
@@
       (at 172.72 269.24 0)
       (effects
+        (font
+          (size 1.27 1.27)) hide))
+    (property "Manufacturer" ""
+      (at 172.72 269.24 0)
+      (effects
