File: 05_NFC.kicad_sch (KiCad schematic)
At the start: 3 parts, among them U4 ST25TN01K-AFH5

Commit message: Complete procurement BOM and document component review gates
Parts:
- U4: Manufacturer (none) -> STMicroelectronics
Changed lines of the file:
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@@
+        (font
+          (size 1.27 1.27)) hide))
+    (property "Manufacturer" "STMicroelectronics"
+      (at 231.14 91.44 0)
+      (effects
         (font
           (size 1.27 1.27)) hide))
@@
         (font
           (size 1.27 1.27)) hide))
+    (property "Manufacturer" ""
+      (at 68.58 91.44 0)
+      (effects
+        (font
+          (size 1.27 1.27)) hide))
     (pin "1"
 )
@@
       (at 144.78 91.44 0)
       (effects
+        (font
+          (size 1.27 1.27)) hide))
+    (property "Manufacturer" ""
+      (at 144.78 91.44 0)
+      (effects
