File: SnakeBusinessCard.kicad_pcb (KiCad board)
At the start: 2 copper layers, 85.6 x 54 mm, 136 parts, among them J1 UJC-HP-3-SMT-TR, SW1 UP, SW2 DOWN, SW3 LEFT, SW4 RIGHT, SW5 START, U1 STM32G030K8T6, U2 IS31FL3737-QFLS4-TR, U3 TLV75533PDBVR, U4 ST25TN01K-AFH5, U5 TPD2E2U06DCK

Commit message: Complete procurement BOM and document component review gates
Parts:
- C1, C2, C23, C24: value 1u / 10V X7R -> 1u / 35V X7R
- C10, C12, C20, C21, C22: value 100n / 10V X7R -> 100n / 50V X7R
- C11: value 4.7u / 10V X7R -> 4.7u / 16V
- R10, R11, R12, R13, R14, R15, R23: value 10k -> 10k 1%
- R20, R21: value 2.2k -> 2.2k 1%
- R22: value 100k -> 100k 1%

Commit message: Use Alex Xu throughout the public example
Other:
- board text added: "REV B / AX-01"
- board text added: "XU"
- board text removed: "PARKER"
- board text removed: "REV B / AP-01"
Changed lines of the file:
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@@
 		)
 	)
-	(property "AUTHOR" "Alex Parker")
+	(property "AUTHOR" "Alex Xu")
 	(property "DESIGN_STAGE" "PLACEMENT REVIEW")
 	(footprint "SnakeCard:Kingbright_APT1608SURCK"
@@
 		)
 	)
-	(gr_text "PARKER"
+	(gr_text "XU"
 		(at 111 97 0)
 		(layer "F.SilkS")
@@
 		)
 	)
-	(gr_text "REV B / AP-01"
+	(gr_text "REV B / AX-01"
 		(at 129.6 131 0)
 		(layer "B.SilkS")
